File: Pin_13_LED.kicad_sch (KiCad schematic)
At the start: 3 parts, among them U2 LMV358IDGKR

Commit message: add packages
Parts:
- D3: footprint ~ -> LED_SMD:LED_0603_1608Metric
- R4: footprint ~ -> Resistor_SMD:R_0603_1608Metric
- U2: footprint ~ -> Package_SO:HVSSOP-8-1EP_3x3mm_P0.65mm_EP1.57x1.89mm
Changed lines of the file:
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@@
       (effects (font (size 1.524 1.524)) (justify left))
     )
-    (property "Footprint" "~" (at 143.51 101.6 0)
-      (effects (font (size 1.524 1.524)))
+    (property "Footprint" "Package_SO:HVSSOP-8-1EP_3x3mm_P0.65mm_EP1.57x1.89mm" (at 143.51 101.6 0)
+      (effects (font (size 1.524 1.524)) hide)
     )
     (property "Datasheet" "http://www.ti.com/lit/ds/symlink/lmv358.pdf" (at 143.51 101.6 0)
@@
       (effects (font (size 1.27 1.27)))
     )
-    (property "Footprint" "~" (at 176.53 111.76 0)
-      (effects (font (size 1.524 1.524)))
+    (property "Footprint" "LED_SMD:LED_0603_1608Metric" (at 176.53 111.76 0)
+      (effects (font (size 1.524 1.524)) hide)
     )
     (property "Datasheet" "http://www.osram-os.com/Graphics/XPic9/00078860_0.pdf" (at 176.53 111.76 0)
@@
       (effects (font (size 1.016 1.016)))
     )
-    (property "Footprint" "~" (at 165.1 103.378 90)
-      (effects (font (size 0.762 0.762)))
+    (property "Footprint" "Resistor_SMD:R_0603_1608Metric" (at 165.1 103.378 90)
+      (effects (font (size 0.762 0.762)) hide)
     )
     (property "Datasheet" "http://www.yageo.com/pdf/Pu-RC0805_51_PbFree_L_2.pdf" (at 165.1 101.6 0)
