File: ATMEGA16U2.kicad_sch (KiCad schematic)
At the start: 16 parts, among them U4 ATMEGA16U2-MU, X1 FOXSLF/160-20

Commit message: update power symbols
Parts:
- D4: symbol Device:D_Filled -> Device:D_Schottky_Small
- JP2: now not fitted; now left out of the parts list
Changed lines of the file:
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@@
     (stroke (width 0) (type default))
   )
-  (wire (pts (xy 110.49 48.26) (xy 110.49 39.37))
+  (wire (pts (xy 110.49 38.1) (xy 110.49 48.26))
     (stroke (width 0) (type default))
   )
@@
     (stroke (width 0) (type default))
   )
-  (wire (pts (xy 110.49 24.13) (xy 110.49 31.75))
+  (wire (pts (xy 110.49 24.13) (xy 110.49 33.02))
     (stroke (width 0) (type default))
   )
@@
     )
   )
-  (symbol (lib_id "Device:D_Filled") (at 110.49 35.56 90) (unit 1)
+  (symbol (lib_id "Device:D_Schottky_Small") (at 110.49 35.56 90) (unit 1)
     (in_bom yes) (on_board yes) (dnp no)
     (property "Reference" "D4" (at 107.95 35.56 0)
@@
       (effects (font (size 1.016 1.016)))
     )
-    (property "Footprint" "Diode_SMD:D_SMA" (at 110.49 35.56 0)
-      (effects (font (size 1.524 1.524)) hide)
-    )
-    (property "Datasheet" "http://www.diodes.com/_files/datasheets/ds30086.pdf" (at 110.49 35.56 0)
-      (effects (font (size 1.524 1.524)) hide)
+    (property "Footprint" "Diode_SMD:D_SMA" (at 110.49 35.56 90)
+      (effects (font (size 1.27 1.27)) hide)
+    )
+    (property "Datasheet" "~" (at 110.49 35.56 90)
+      (effects (font (size 1.27 1.27)) hide)
     )
     (property "Characteristics" "DIODE GEN PURP 100V 300MA SOD123" (at 110.49 35.56 0)
@@
   )
   (symbol (lib_id "Connector_Generic:Conn_02x02_Odd_Even") (at 200.66 45.72 0) (mirror y) (unit 1)
-    (in_bom yes) (on_board yes) (dnp no)
+    (in_bom no) (on_board yes) (dnp yes)
     (property "Reference" "JP2" (at 199.39 43.18 0)
       (effects (font (size 1.27 1.27)))
@@
     )
   )
-  (symbol (lib_id "power:+5V") (at 218.44 127 0) (unit 1)
-    (in_bom yes) (on_board yes) (dnp no)
-    (property "Reference" "#PWR031" (at 218.44 124.714 0)
-      (effects (font (size 0.508 0.508)) hide)
-    )
-    (property "Value" "5V_LDO" (at 218.44 123.825 0)
-      (effects (font (size 1.016 1.016)))
-    )
-    (property "Footprint" "~" (at 218.44 127 0)
-      (effects (font (size 1.27 1.27)) hide)
-    )
-    (property "Datasheet" "~" (at 218.44 127 0)
-      (effects (font (size 1.27 1.27)) hide)
-    )
-    (pin "1")
-    (instances
-      (project "Arduino_Uno_R3_From_Scratch"
-        (path "/e37abd6a-5ce5-42fd-a932-3d77ac2d4dc6/00000000-0000-0000-0000-000055dd0855"
-          (reference "#PWR031") (unit 1)
-        )
-      )
-    )
-  )
   (symbol (lib_id "Device:C") (at 87.63 83.82 90) (unit 1)
     (in_bom yes) (on_board yes) (dnp no)
@@
   )
   (symbol (lib_id "Device:R") (at 100.33 35.56 180) (unit 1)
-    (in_bom yes) (on_board yes) (dnp no)
+    (in_bom yes) (on_board no) (dnp no)
     (property "Reference" "R7" (at 98.298 35.56 90)
       (effects (font (size 1.016 1.016)))
@@
     )
   )
+  (symbol (lib_id "power:+5V") (at 87.63 93.98 0) (unit 1)
+    (in_bom yes) (on_board yes) (dnp no)
+    (property "Reference" "#PWR0201" (at 87.63 97.79 0)
+      (effects (font (size 1.27 1.27)) hide)
+    )
+    (property "Value" "+5V" (at 87.63 90.17 0)
+      (effects (font (size 1.016 1.016)))
+    )
+    (property "Footprint" "" (at 87.63 93.98 0)
+      (effects (font (size 1.27 1.27)) hide)
+    )
+    (property "Datasheet" "" (at 87.63 93.98 0)
+      (effects (font (size 1.27 1.27)) hide)
+    )
+    (pin "1")
+    (instances
+      (project "Arduino_Uno_R3_From_Scratch"
+        (path "/e37abd6a-5ce5-42fd-a932-3d77ac2d4dc6/00000000-0000-0000-0000-000055ccfea2"
+          (reference "#PWR0201") (unit 1)
+        )
+        (path "/e37abd6a-5ce5-42fd-a932-3d77ac2d4dc6/00000000-0000-0000-0000-000055d9f413"
+          (reference "#PWR0303") (unit 1)
+        )
+        (path "/e37abd6a-5ce5-42fd-a932-3d77ac2d4dc6/00000000-0000-0000-0000-000055d0d7e6"
+          (reference "#PWR0408") (unit 1)
+        )
+        (path "/e37abd6a-5ce5-42fd-a932-3d77ac2d4dc6/00000000-0000-0000-0000-000055dd0855"
+          (reference "#PWR0506") (unit 1)
+        )
+      )
+    )
+  )
   (symbol (lib_id "power:VCC") (at 105.41 106.68 0) (unit 1)
     (in_bom yes) (on_board yes) (dnp no)
-    (property "Reference" "#PWR032" (at 105.41 104.394 0)
-      (effects (font (size 0.508 0.508)) hide)
-    )
-    (property "Value" "USBVCC" (at 105.41 103.505 0)
-      (effects (font (size 1.016 1.016)))
-    )
-    (property "Footprint" "~" (at 105.41 106.68 0)
-      (effects (font (size 1.27 1.27)) hide)
-    )
-    (property "Datasheet" "~" (at 105.41 106.68 0)
-      (effects (font (size 1.27 1.27)) hide)
-    )
-    (pin "1")
-    (instances
-      (project "Arduino_Uno_R3_From_Scratch"
-        (path "/e37abd6a-5ce5-42fd-a932-3d77ac2d4dc6/00000000-0000-0000-0000-000055dd0855"
-          (reference "#PWR032") (unit 1)
-        )
-      )
-    )
-  )
-  (symbol (lib_id "power:+5V") (at 87.63 93.98 0) (unit 1)
-    (in_bom yes) (on_board yes) (dnp no)
-    (property "Reference" "#PWR033" (at 87.63 91.694 0)
-      (effects (font (size 0.508 0.508)) hide)
-    )
-    (property "Value" "5V_LDO" (at 87.63 90.805 0)
-      (effects (font (size 1.016 1.016)))
-    )
-    (property "Footprint" "~" (at 87.63 93.98 0)
-      (effects (font (size 1.27 1.27)) hide)
-    )
-    (property "Datasheet" "~" (at 87.63 93.98 0)
-      (effects (font (size 1.27 1.27)) hide)
-    )
-    (pin "1")
-    (instances
-      (project "Arduino_Uno_R3_From_Scratch"
-        (path "/e37abd6a-5ce5-42fd-a932-3d77ac2d4dc6/00000000-0000-0000-0000-000055dd0855"
-          (reference "#PWR033") (unit 1)
+    (property "Reference" "#PWR0202" (at 105.41 110.49 0)
+      (effects (font (size 1.27 1.27)) hide)
+    )
+    (property "Value" "VCC" (at 105.41 102.87 0)
+      (effects (font (size 1.016 1.016)))
+    )
+    (property "Footprint" "" (at 105.41 106.68 0)
+      (effects (font (size 1.27 1.27)) hide)
+    )
+    (property "Datasheet" "" (at 105.41 106.68 0)
+      (effects (font (size 1.27 1.27)) hide)
+    )
+    (pin "1")
+    (instances
+      (project "Arduino_Uno_R3_From_Scratch"
+        (path "/e37abd6a-5ce5-42fd-a932-3d77ac2d4dc6/00000000-0000-0000-0000-000055ccfea2"
+          (reference "#PWR0202") (unit 1)
+        )
+        (path "/e37abd6a-5ce5-42fd-a932-3d77ac2d4dc6/00000000-0000-0000-0000-000055d9f413"
+          (reference "#PWR0301") (unit 1)
+        )
+        (path "/e37abd6a-5ce5-42fd-a932-3d77ac2d4dc6/00000000-0000-0000-0000-000055d0d7e6"
+          (reference "#PWR0409") (unit 1)
+        )
+        (path "/e37abd6a-5ce5-42fd-a932-3d77ac2d4dc6/00000000-0000-0000-0000-000055dd0855"
+          (reference "#PWR0503") (unit 1)
         )
       )
@@
   (symbol (lib_id "power:+5V") (at 100.33 20.32 0) (unit 1)
     (in_bom yes) (on_board yes) (dnp no)
-    (property "Reference" "#PWR034" (at 100.33 18.034 0)
-      (effects (font (size 0.508 0.508)) hide)
-    )
-    (property "Value" "5V_LDO" (at 100.33 17.272 0)
-      (effects (font (size 1.016 1.016)))
-    )
-    (property "Footprint" "~" (at 100.33 20.32 0)
-      (effects (font (size 1.27 1.27)) hide)
-    )
-    (property "Datasheet" "~" (at 100.33 20.32 0)
-      (effects (font (size 1.27 1.27)) hide)
-    )
-    (pin "1")
-    (instances
-      (project "Arduino_Uno_R3_From_Scratch"
-        (path "/e37abd6a-5ce5-42fd-a932-3d77ac2d4dc6/00000000-0000-0000-0000-000055dd0855"
-          (reference "#PWR034") (unit 1)
-        )
-      )
+    (property "Reference" "#PWR0201" (at 100.33 24.13 0)
+      (effects (font (size 1.27 1.27)) hide)
+    )
+    (property "Value" "+5V" (at 100.33 16.51 0)
+      (effects (font (size 1.016 1.016)))
+    )
+    (property "Footprint" "" (at 100.33 20.32 0)
+      (effects (font (size 1.27 1.27)) hide)
+    )
+    (property "Datasheet" "" (at 100.33 20.32 0)
+      (effects (font (size 1.27 1.27)) hide)
+    )
+    (pin "1")
+    (instances
+      (project "Arduino_Uno_R3_From_Scratch"
+        (path "/e37abd6a-5ce5-42fd-a932-3d77ac2d4dc6/00000000-0000-0000-0000-000055ccfea2"
+          (reference "#PWR0201") (unit 1)
+        )
+        (path "/e37abd6a-5ce5-42fd-a932-3d77ac2d4dc6/00000000-0000-0000-0000-000055d9f413"
+          (reference "#PWR0303") (unit 1)
+        )
+        (path "/e37abd6a-5ce5-42fd-a932-3d77ac2d4dc6/00000000-0000-0000-0000-000055d0d7e6"
+          (reference "#PWR0408") (unit 1)
+        )
+        (path "/e37abd6a-5ce5-42fd-a932-3d77ac2d4dc6/00000000-0000-0000-0000-000055dd0855"
+          (reference "#PWR0502") (unit 1)
+        )
+      )
+    )
+  )
+  (symbol (lib_id "power:+5V") (at 218.44 127 0) (unit 1)
+    (in_bom yes) (on_board yes) (dnp no)
+    (property "Reference" "#PWR0201" (at 218.44 130.81 0)
+      (effects (font (size 1.27 1.27)) hide)
+    )
+    (property "Value" "+5V" (at 218.44 123.19 0)
+      (effects (font (size 1.016 1.016)))
+    )
+    (property "Footprint" "" (at 218.44 127 0)
+      (effects (font (size 1.27 1.27)) hide)
+    )
+    (property "Datasheet" "" (at 218.44 127 0)
+      (effects (font (size 1.27 1.27)) hide)
+    )
+    (pin "1")
+    (instances
+      (project "Arduino_Uno_R3_From_Scratch"
+        (path "/e37abd6a-5ce5-42fd-a932-3d77ac2d4dc6/00000000-0000-0000-0000-000055ccfea2"
+          (reference "#PWR0201") (unit 1)
+        )
+        (path "/e37abd6a-5ce5-42fd-a932-3d77ac2d4dc6/00000000-0000-0000-0000-000055d9f413"
+          (reference "#PWR0303") (unit 1)
+        )
+        (path "/e37abd6a-5ce5-42fd-a932-3d77ac2d4dc6/00000000-0000-0000-0000-000055d0d7e6"
+          (reference "#PWR0408") (unit 1)
+        )
+        (path "/e37abd6a-5ce5-42fd-a932-3d77ac2d4dc6/00000000-0000-0000-0000-000055dd0855"
+          (reference "#PWR0504") (unit 1)
+        )
+      )
