File: ATMEGA328P.kicad_sch (KiCad schematic)
At the start: 14 parts, among them SW1 RESET_SWITCH, U5 ATMEGA328P, X2 CSTCE16MOV53-R0

Commit message: add packages
Parts:
- C11, C14, C15: footprint ~ -> Capacitor_SMD:C_0603_1608Metric
- D7: footprint ~ -> Diode_SMD:D_SMA
- ICSP2: footprint ~ -> Connector_PinHeader_2.54mm:PinHeader_2x03_P2.54mm_Vertical
- R12, R13, R14, R15, R16, R17: footprint ~ -> Resistor_SMD:R_0603_1608Metric
- SW1: footprint (none) -> Button_Switch_SMD:SW_SPST_PTS645
- U5: footprint ~ -> Package_QFP:TQFP-32_7x7mm_P0.8mm
- X2: footprint ~ -> Crystal:Crystal_AT310_D3.0mm_L10.0mm_Horizontal_1EP_style1
Changed lines of the file:
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@@
       (effects (font (size 1.524 1.524)))
     )
-    (property "Footprint" "~" (at 176.53 57.15 0)
-      (effects (font (size 1.524 1.524)))
+    (property "Footprint" "Package_QFP:TQFP-32_7x7mm_P0.8mm" (at 176.53 57.15 0)
+      (effects (font (size 1.524 1.524)) hide)
     )
     (property "Datasheet" "http://www.atmel.com/images/Atmel-8271-8-bit-AVR-Microcontroller-ATmega48A-48PA-88A-88PA-168A-168PA-328-328P_datasheet_Complete.pdf" (at 176.53 57.15 0)
@@
       (effects (font (size 1.016 1.016)))
     )
-    (property "Footprint" "~" (at 37.592 49.53 90)
-      (effects (font (size 0.762 0.762)))
+    (property "Footprint" "Resistor_SMD:R_0603_1608Metric" (at 37.592 49.53 90)
+      (effects (font (size 0.762 0.762)) hide)
     )
     (property "Datasheet" "http://images.ihscontent.net/vipimages/VipMasterIC/IC/VISH/VISHS75859/VISHS75859-1.pdf" (at 39.37 49.53 0)
@@
       (effects (font (size 1.016 1.016)))
     )
-    (property "Footprint" "~" (at 95.25 21.59 0)
-      (effects (font (size 1.524 1.524)))
+    (property "Footprint" "Connector_PinHeader_2.54mm:PinHeader_2x03_P2.54mm_Vertical" (at 95.25 21.59 0)
+      (effects (font (size 1.524 1.524)) hide)
     )
     (property "Datasheet" "http://cdn.harwin.com/pdfs/M20-998.pdf" (at 95.25 21.59 0)
@@
       (effects (font (size 1.016 1.016)))
     )
-    (property "Footprint" "~" (at 134.62 30.48 0)
-      (effects (font (size 1.524 1.524)))
+    (property "Footprint" "Diode_SMD:D_SMA" (at 134.62 30.48 0)
+      (effects (font (size 1.524 1.524)) hide)
     )
     (property "Datasheet" "http://www.diodes.com/_files/datasheets/ds30086.pdf" (at 134.62 30.48 0)
@@
       (effects (font (size 1.524 1.524)))
     )
-    (property "Footprint" "" (at 86.36 50.8 0)
-      (effects (font (size 1.524 1.524)))
+    (property "Footprint" "Button_Switch_SMD:SW_SPST_PTS645" (at 86.36 50.8 0)
+      (effects (font (size 1.524 1.524)) hide)
     )
     (property "Datasheet" "http://industrial.panasonic.com/www-data/pdf/ATK0000/ATK0000CE28.pdf" (at 86.36 50.8 0)
@@
       (effects (font (size 1.016 1.016)))
     )
-    (property "Footprint" "~" (at 68.58 39.878 90)
-      (effects (font (size 0.762 0.762)))
+    (property "Footprint" "Resistor_SMD:R_0603_1608Metric" (at 68.58 39.878 90)
+      (effects (font (size 0.762 0.762)) hide)
     )
     (property "Datasheet" "http://industrial.panasonic.com/www-cgi/jvcr13pz.cgi?E+PZ+3+AOA0001+ERJ6GEY0R00V+7+WW" (at 68.58 38.1 0)
@@
       (effects (font (size 1.016 1.016)) (justify right))
     )
-    (property "Footprint" "~" (at 133.35 64.77 0)
-      (effects (font (size 1.524 1.524)))
+    (property "Footprint" "Crystal:Crystal_AT310_D3.0mm_L10.0mm_Horizontal_1EP_style1" (at 133.35 64.77 0)
+      (effects (font (size 1.524 1.524)) hide)
     )
     (property "Datasheet" "http://www.murata.com/~/media/webrenewal/support/library/catalog/products/timingdevice/ceralock/p16e.ashx" (at 133.35 64.77 0)
@@
       (effects (font (size 1.016 1.016)) (justify left))
     )
-    (property "Footprint" "~" (at 130.5052 109.22 0)
-      (effects (font (size 0.762 0.762)))
+    (property "Footprint" "Capacitor_SMD:C_0603_1608Metric" (at 130.5052 109.22 0)
+      (effects (font (size 0.762 0.762)) hide)
     )
     (property "Datasheet" "http://images.ihscontent.net/vipimages/VipMasterIC/IC/KEME/KEMES10043/KEMES10043-1.pdf" (at 129.54 105.41 0)
@@
       (effects (font (size 1.016 1.016)) (justify left))
     )
-    (property "Footprint" "~" (at 143.2052 133.35 0)
-      (effects (font (size 0.762 0.762)))
+    (property "Footprint" "Capacitor_SMD:C_0603_1608Metric" (at 143.2052 133.35 0)
+      (effects (font (size 0.762 0.762)) hide)
     )
     (property "Datasheet" "http://images.ihscontent.net/vipimages/VipMasterIC/IC/KEME/KEMES10043/KEMES10043-1.pdf" (at 142.24 129.54 0)
@@
       (effects (font (size 1.016 1.016)))
     )
-    (property "Footprint" "~" (at 126.238 30.48 90)
-      (effects (font (size 0.762 0.762)))
+    (property "Footprint" "Resistor_SMD:R_0603_1608Metric" (at 126.238 30.48 90)
+      (effects (font (size 0.762 0.762)) hide)
     )
     (property "Datasheet" "http://images.ihscontent.net/vipimages/VipMasterIC/IC/VISH/VISHS75859/VISHS75859-1.pdf" (at 124.46 30.48 0)
@@
       (effects (font (size 1.016 1.016)))
     )
-    (property "Footprint" "~" (at 68.58 145.288 90)
-      (effects (font (size 0.762 0.762)))
+    (property "Footprint" "Resistor_SMD:R_0603_1608Metric" (at 68.58 145.288 90)
+      (effects (font (size 0.762 0.762)) hide)
     )
     (property "Datasheet" "http://images.ihscontent.net/vipimages/VipMasterIC/IC/VISH/VISHS75859/VISHS75859-1.pdf" (at 68.58 143.51 0)
@@
       (effects (font (size 1.016 1.016)))
     )
-    (property "Footprint" "~" (at 68.58 151.638 90)
-      (effects (font (size 0.762 0.762)))
+    (property "Footprint" "Resistor_SMD:R_0603_1608Metric" (at 68.58 151.638 90)
+      (effects (font (size 0.762 0.762)) hide)
     )
     (property "Datasheet" "http://images.ihscontent.net/vipimages/VipMasterIC/IC/VISH/VISHS75859/VISHS75859-1.pdf" (at 68.58 149.86 0)
@@
       (effects (font (size 1.016 1.016)))
     )
-    (property "Footprint" "~" (at 55.88 37.1348 0)
-      (effects (font (size 0.762 0.762)))
+    (property "Footprint" "Capacitor_SMD:C_0603_1608Metric" (at 55.88 37.1348 0)
+      (effects (font (size 0.762 0.762)) hide)
     )
     (property "Datasheet" "http://images.ihscontent.net/vipimages/VipMasterIC/IC/KEME/KEMES10043/KEMES10043-1.pdf" (at 52.07 38.1 0)
@@
       (effects (font (size 1.016 1.016)))
     )
-    (property "Footprint" "~" (at 141.732 64.77 90)
-      (effects (font (size 0.762 0.762)))
+    (property "Footprint" "Resistor_SMD:R_0603_1608Metric" (at 141.732 64.77 90)
+      (effects (font (size 0.762 0.762)) hide)
     )
     (property "Datasheet" "http://www.vishay.com/docs/20035/dcrcwe3.pdf" (at 143.51 64.77 0)

Commit message: change power symbols and Arduino header
Parts:
- removed ICSP2: M20-9980346, Connector_PinHeader_2.54mm:PinHeader_2x03_P2.54mm_Vertical, symbol Connector_Generic:Conn_02x03_Odd_Even
Connections:
- net 328P_ICSP_MISO renamed ARD_DIG12/SPI_MISO
- net 328P_ICSP_MOSI renamed ARD_DIG11/SPI_MOSI
- net 328P_ICSP_SCK renamed ARD_DIG13/SPI_SCK
- net 328P_RESET renamed +5V
- net +5V: now also C15.1, R16.2, U5.20 (AVCC), U5.7 (VCC)
- removed net 5V_LDO: C15.1, D7.2 (A), R16.2, U5.20 (AVCC), U5.7 (VCC)
- new net 328P_ICSP_VIN: D7.2 (A)
Other:
- moved on the sheet: D7

Commit message: update power symbols
Parts:
- removed D7: 1N4148W-7-F, Diode_SMD:D_SMA, symbol Device:D_Filled
Connections:
- net +5V: no longer R13.2, R16.1, SW1.3, SW1.4, U5.1 (~{RESET})
- new net 328P_RESET: R13.2, R16.1, SW1.3, SW1.4, U5.1 (~{RESET})
Changed lines of the file:
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@@
   (junction (at 142.24 114.3) (diameter 0) (color 0 0 0 0)
   )
-  (junction (at 124.46 19.05) (diameter 0) (color 0 0 0 0)
-  )
-  (junction (at 134.62 38.1) (diameter 0) (color 0 0 0 0)
-  )
   (junction (at 39.37 38.1) (diameter 0) (color 0 0 0 0)
   )
@@
     (stroke (width 0) (type default))
   )
-  (wire (pts (xy 124.46 38.1) (xy 134.62 38.1))
+  (wire (pts (xy 124.46 38.1) (xy 143.51 38.1))
     (stroke (width 0) (type default))
   )
@@
     (stroke (width 0) (type default))
   )
-  (wire (pts (xy 143.51 19.05) (xy 237.49 19.05))
+  (wire (pts (xy 143.51 19.05) (xy 146.05 19.05))
     (stroke (width 0) (type default))
   )
@@
     (stroke (width 0) (type default))
   )
-  (wire (pts (xy 124.46 19.05) (xy 124.46 26.67))
+  (wire (pts (xy 124.46 21.59) (xy 124.46 26.67))
     (stroke (width 0) (type default))
   )
@@
     (stroke (width 0) (type default))
   )
-  (wire (pts (xy 116.84 19.05) (xy 124.46 19.05))
-    (stroke (width 0) (type default))
-  )
   (wire (pts (xy 86.36 38.1) (xy 124.46 38.1))
     (stroke (width 0) (type default))
@@
     (stroke (width 0) (type default))
   )
-  (wire (pts (xy 99.06 19.05) (xy 109.22 19.05))
-    (stroke (width 0) (type default))
-  )
   (wire (pts (xy 142.24 119.38) (xy 142.24 125.73))
     (stroke (width 0) (type default))
@@
     (stroke (width 0) (type default))
   )
-  (wire (pts (xy 134.62 38.1) (xy 143.51 38.1))
-    (stroke (width 0) (type default))
-  )
   (wire (pts (xy 31.75 38.1) (xy 39.37 38.1))
     (stroke (width 0) (type default))
@@
     (stroke (width 0) (type default))
   )
-  (wire (pts (xy 124.46 19.05) (xy 134.62 19.05))
-    (stroke (width 0) (type default))
-  )
   (wire (pts (xy 217.17 149.86) (xy 237.49 149.86))
     (stroke (width 0) (type default))
@@
     (stroke (width 0) (type default))
   )
-  (wire (pts (xy 134.62 19.05) (xy 134.62 38.1))
-    (stroke (width 0) (type default))
-  )
   (wire (pts (xy 209.55 124.46) (xy 237.49 124.46))
     (stroke (width 0) (type default))
@@
   )
   (wire (pts (xy 72.39 38.1) (xy 86.36 38.1))
-    (stroke (width 0) (type default))
-  )
-  (wire (pts (xy 124.46 16.51) (xy 124.46 19.05))
     (stroke (width 0) (type default))
   )
@@
     (effects (font (size 1.016 1.016)) (justify left))
   )
-  (hierarchical_label "328P_RESET" (shape input) (at 237.49 19.05 0) (fields_autoplaced)
+  (hierarchical_label "328P_RESET" (shape input) (at 146.05 19.05 0) (fields_autoplaced)
     (effects (font (size 1.016 1.016)) (justify left))
   )
@@
   (hierarchical_label "ARD_AN4/SDA" (shape input) (at 237.49 87.63 0) (fields_autoplaced)
     (effects (font (size 1.016 1.016)) (justify left))
-  )
-  (hierarchical_label "328P_ICSP_VIN" (shape input) (at 99.06 19.05 180) (fields_autoplaced)
-    (effects (font (size 1.016 1.016)) (justify right))
   )
   (hierarchical_label "ARD_DIG5" (shape input) (at 237.49 129.54 0) (fields_autoplaced)
@@
     )
   )
-  (symbol (lib_id "Device:D_Filled") (at 113.03 19.05 0) (mirror y) (unit 1)
-    (in_bom yes) (on_board yes) (dnp no)
-    (property "Reference" "D7" (at 113.03 16.51 0)
-      (effects (font (size 1.016 1.016)))
-    )
-    (property "Value" "1N4148W-7-F" (at 113.03 21.59 0)
-      (effects (font (size 1.016 1.016)))
-    )
-    (property "Footprint" "Diode_SMD:D_SMA" (at 113.03 19.05 0)
-      (effects (font (size 1.524 1.524)) hide)
-    )
-    (property "Datasheet" "http://www.diodes.com/_files/datasheets/ds30086.pdf" (at 113.03 19.05 0)
-      (effects (font (size 1.524 1.524)) hide)
-    )
-    (property "Characteristics" "DIODE GEN PURP 100V 300MA SOD123" (at 113.03 19.05 0)
-      (effects (font (size 1.524 1.524)) hide)
-    )
-    (property "Description" "ATMEGA328P ICSP Reset Voltage Spike Protection" (at 113.03 19.05 0)
-      (effects (font (size 1.524 1.524)) hide)
-    )
-    (property "MFN" "Diodes Inc" (at 113.03 19.05 0)
-      (effects (font (size 1.524 1.524)) hide)
-    )
-    (property "Package ID" "SOD123" (at 113.03 19.05 0)
-      (effects (font (size 1.524 1.524)) hide)
-    )
-    (property "Source" "ANY" (at 113.03 19.05 0)
-      (effects (font (size 1.524 1.524)) hide)
-    )
-    (property "Critical" "N" (at 113.03 19.05 0)
-      (effects (font (size 1.524 1.524)) hide)
-    )
-    (property "Subsystem" "328P_Sub" (at 113.03 19.05 0)
-      (effects (font (size 1.524 1.524)) hide)
-    )
-    (property "Notes" "~" (at 113.03 19.05 0)
-      (effects (font (size 1.524 1.524)) hide)
-    )
-    (property "MPN" "1N4148W-7-F" (at 113.03 19.05 0)
-      (effects (font (size 1.27 1.27)) hide)
-    )
-    (pin "1")
-    (pin "2")
-    (instances
-      (project "Arduino_Uno_R3_From_Scratch"
-        (path "/e37abd6a-5ce5-42fd-a932-3d77ac2d4dc6/00000000-0000-0000-0000-000055e89ce4"
-          (reference "D7") (unit 1)
-        )
-        (path "/e37abd6a-5ce5-42fd-a932-3d77ac2d4dc6"
-          (reference "D7") (unit 1)
-        )
-      )
-    )
-  )
   (symbol (lib_id "Arduino_Uno_R3_From_Scratch:RESET_SWITCH") (at 86.36 50.8 90) (unit 1)
     (in_bom yes) (on_board yes) (dnp no)
@@
     )
   )
-  (symbol (lib_id "power:+5V") (at 124.46 16.51 0) (unit 1)
-    (in_bom yes) (on_board yes) (dnp no)
-    (property "Reference" "#PWR041" (at 124.46 14.224 0)
-      (effects (font (size 0.508 0.508)) hide)
-    )
-    (property "Value" "5V_LDO" (at 124.46 13.462 0)
-      (effects (font (size 0.762 0.762)))
-    )
-    (property "Footprint" "~" (at 124.46 16.51 0)
-      (effects (font (size 1.27 1.27)) hide)
-    )
-    (property "Datasheet" "~" (at 124.46 16.51 0)
-      (effects (font (size 1.27 1.27)) hide)
-    )
-    (pin "1")
-    (instances
-      (project "Arduino_Uno_R3_From_Scratch"
-        (path "/e37abd6a-5ce5-42fd-a932-3d77ac2d4dc6/00000000-0000-0000-0000-000055e89ce4"
-          (reference "#PWR041") (unit 1)
-        )
-      )
-    )
-  )
-  (symbol (lib_id "power:+5V") (at 142.24 109.22 0) (unit 1)
-    (in_bom yes) (on_board yes) (dnp no)
-    (property "Reference" "#PWR042" (at 142.24 106.934 0)
-      (effects (font (size 0.508 0.508)) hide)
-    )
-    (property "Value" "5V_LDO" (at 142.24 106.172 0)
-      (effects (font (size 1.016 1.016)))
-    )
-    (property "Footprint" "~" (at 142.24 109.22 0)
-      (effects (font (size 1.27 1.27)) hide)
-    )
-    (property "Datasheet" "~" (at 142.24 109.22 0)
-      (effects (font (size 1.27 1.27)) hide)
-    )
-    (pin "1")
-    (instances
-      (project "Arduino_Uno_R3_From_Scratch"
-        (path "/e37abd6a-5ce5-42fd-a932-3d77ac2d4dc6/00000000-0000-0000-0000-000055e89ce4"
-          (reference "#PWR042") (unit 1)
-        )
-      )
-    )
-  )
   (symbol (lib_id "Device:R") (at 68.58 38.1 90) (unit 1)
     (in_bom yes) (on_board yes) (dnp no)
@@
         )
       )
+    )
+  )
+  (symbol (lib_id "power:+5V") (at 124.46 21.59 0) (unit 1)
+    (in_bom yes) (on_board yes) (dnp no)
+    (property "Reference" "#PWR0201" (at 124.46 25.4 0)
+      (effects (font (size 1.27 1.27)) hide)
+    )
+    (property "Value" "+5V" (at 124.46 17.78 0)
+      (effects (font (size 1.016 1.016)))
+    )
+    (property "Footprint" "" (at 124.46 21.59 0)
+      (effects (font (size 1.27 1.27)) hide)
+    )
+    (property "Datasheet" "" (at 124.46 21.59 0)
+      (effects (font (size 1.27 1.27)) hide)
+    )
+    (pin "1")
+    (instances
+      (project "Arduino_Uno_R3_From_Scratch"
+        (path "/e37abd6a-5ce5-42fd-a932-3d77ac2d4dc6/00000000-0000-0000-0000-000055ccfea2"
+          (reference "#PWR0201") (unit 1)
+        )
+        (path "/e37abd6a-5ce5-42fd-a932-3d77ac2d4dc6/00000000-0000-0000-0000-000055d9f413"
+          (reference "#PWR0303") (unit 1)
+        )
+        (path "/e37abd6a-5ce5-42fd-a932-3d77ac2d4dc6/00000000-0000-0000-0000-000055d0d7e6"
+          (reference "#PWR0408") (unit 1)
+        )
+        (path "/e37abd6a-5ce5-42fd-a932-3d77ac2d4dc6/00000000-0000-0000-0000-000055e89ce4"
+          (reference "#PWR0602") (unit 1)
+        )
+      )
+    )
+  )
+  (symbol (lib_id "power:+5V") (at 142.24 109.22 0) (unit 1)
+    (in_bom yes) (on_board yes) (dnp no)
+    (property "Reference" "#PWR0201" (at 142.24 113.03 0)
+      (effects (font (size 1.27 1.27)) hide)
+    )
+    (property "Value" "+5V" (at 142.24 105.41 0)
+      (effects (font (size 1.016 1.016)))
+    )
+    (property "Footprint" "" (at 142.24 109.22 0)
+      (effects (font (size 1.27 1.27)) hide)
+    )
+    (property "Datasheet" "" (at 142.24 109.22 0)
+      (effects (font (size 1.27 1.27)) hide)
+    )
+    (pin "1")
+    (instances
+      (project "Arduino_Uno_R3_From_Scratch"
+        (path "/e37abd6a-5ce5-42fd-a932-3d77ac2d4dc6/00000000-0000-0000-0000-000055ccfea2"
+          (reference "#PWR0201") (unit 1)
+        )
+        (path "/e37abd6a-5ce5-42fd-a932-3d77ac2d4dc6/00000000-0000-0000-0000-000055d9f413"
+          (reference "#PWR0303") (unit 1)
+        )
+        (path "/e37abd6a-5ce5-42fd-a932-3d77ac2d4dc6/00000000-0000-0000-0000-000055d0d7e6"
+          (reference "#PWR0408") (unit 1)
+        )
+        (path "/e37abd6a-5ce5-42fd-a932-3d77ac2d4dc6/00000000-0000-0000-0000-000055e89ce4"
+          (reference "#PWR0603") (unit 1)
+        )
+      )
