File: USB_Interface.kicad_sch (KiCad schematic)
At the start: 7 parts, among them J1 USB_TYPE_B

Commit message: add packages
Parts:
- FB1: footprint ~ -> Inductor_SMD:L_0805_2012Metric
- J1: footprint ~ -> Connector_USB:USB_B_Lumberg_2411_02_Horizontal
- MF-MSMF050-2: footprint ~ -> Resistor_SMD:R_0805_2012Metric
- R5, R6, VR1, VR2: footprint ~ -> Resistor_SMD:R_0603_1608Metric
Changed lines of the file:
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@@
       (effects (font (size 1.27 1.27)))
     )
-    (property "Footprint" "~" (at 173.99 76.2 0)
-      (effects (font (size 1.524 1.524)))
+    (property "Footprint" "Resistor_SMD:R_0805_2012Metric" (at 173.99 76.2 0)
+      (effects (font (size 1.524 1.524)) hide)
     )
     (property "Datasheet" "http://www.bourns.com/data/global/pdfs/mfmsmf.pdf" (at 173.99 76.2 0)
@@
       (effects (font (size 1.016 1.016)))
     )
-    (property "Footprint" "~" (at 173.99 88.138 90)
-      (effects (font (size 0.762 0.762)))
+    (property "Footprint" "Resistor_SMD:R_0603_1608Metric" (at 173.99 88.138 90)
+      (effects (font (size 0.762 0.762)) hide)
     )
     (property "Datasheet" "http://www.yageo.com/NewPortal/yageodocoutput?fileName=/pdf/R-Chip/PYu-RC_Group_51_RoHS_L_3.pdf" (at 173.99 86.36 0)
@@
       (effects (font (size 1.016 1.016)))
     )
-    (property "Footprint" "~" (at 136.525 91.44 0)
-      (effects (font (size 1.524 1.524)))
+    (property "Footprint" "Connector_USB:USB_B_Lumberg_2411_02_Horizontal" (at 136.525 91.44 0)
+      (effects (font (size 1.524 1.524)) hide)
     )
     (property "Datasheet" "http://images.ihscontent.net/vipimages/VipMasterIC/IC/TYEL/TYELS17825/TYELS17825-1.pdf" (at 136.525 91.44 0)
@@
       (effects (font (size 1.016 1.016)))
     )
-    (property "Footprint" "~" (at 161.29 100.33 0)
-      (effects (font (size 1.524 1.524)))
+    (property "Footprint" "Resistor_SMD:R_0603_1608Metric" (at 161.29 100.33 0)
+      (effects (font (size 1.524 1.524)) hide)
     )
     (property "Datasheet" "http://www.bourns.com/data/global/pdfs/mlc.pdf" (at 161.29 100.33 0)
@@
       (effects (font (size 1.016 1.016)) (justify left))
     )
-    (property "Footprint" "~" (at 153.67 128.27 0)
-      (effects (font (size 1.524 1.524)))
+    (property "Footprint" "Inductor_SMD:L_0805_2012Metric" (at 153.67 128.27 0)
+      (effects (font (size 1.524 1.524)) hide)
     )
     (property "Datasheet" "http://search.murata.co.jp/Ceramy/image/img/PDF/ENG/L0110S0100BLM21P.pdf" (at 153.67 128.27 0)
@@
       (effects (font (size 1.016 1.016)))
     )
-    (property "Footprint" "~" (at 153.67 100.33 0)
-      (effects (font (size 1.524 1.524)))
+    (property "Footprint" "Resistor_SMD:R_0603_1608Metric" (at 153.67 100.33 0)
+      (effects (font (size 1.524 1.524)) hide)
     )
     (property "Datasheet" "http://www.bourns.com/data/global/pdfs/mlc.pdf" (at 153.67 100.33 0)
@@
       (effects (font (size 1.016 1.016)))
     )
-    (property "Footprint" "~" (at 173.99 91.948 90)
-      (effects (font (size 0.762 0.762)))
+    (property "Footprint" "Resistor_SMD:R_0603_1608Metric" (at 173.99 91.948 90)
+      (effects (font (size 0.762 0.762)) hide)
     )
     (property "Datasheet" "http://www.yageo.com/NewPortal/yageodocoutput?fileName=/pdf/R-Chip/PYu-RC_Group_51_RoHS_L_3.pdf" (at 173.99 90.17 0)

Commit message: change power symbols and Arduino header
Parts:
- J1: footprint Connector_USB:USB_B_Lumberg_2411_02_Horizontal -> Connector_USB:USB_Micro-B_Molex-105017-0001; symbol Arduino_Uno_R3_From_Scratch:USB_TYPE_B -> Connector:USB_B_Micro; Characteristics 4 CONTACT(S), FEMALE, RIGHT ANGLE USB TYPE-B CONNECTOR -> (none); MFN TE Connectivity -> (none); MPN 292304-1 -> (none); Subsystem USB_Cnxn -> (none)
- renumbered MF-MSMF050-2 to F1
Connections:
- net USB_GND: now also J1.5 (GND); no longer J1.4 (GND)
- net at R5.1, VR2.1: now also J1.3 (D+); no longer J1.2 (D-)
- net at R6.1, VR1.1: now also J1.2 (D-); no longer J1.3 (D+)
- net at FB1.1, J1.6 (Shield), VR1.2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: no longer J1.5 (Shield_1)
- net USBVCC renamed VCC
- no-connect marks 0 -> 1
Other:
- moved on the sheet: R5

Commit message: update power symbols
Changed lines of the file:
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@@
   (symbol (lib_id "power:VCC") (at 190.5 71.12 0) (unit 1)
     (in_bom yes) (on_board yes) (dnp no)
-    (property "Reference" "#PWR025" (at 190.5 68.834 0)
-      (effects (font (size 0.508 0.508)) hide)
-    )
-    (property "Value" "USBVCC" (at 190.5 68.072 0)
-      (effects (font (size 0.762 0.762)))
-    )
-    (property "Footprint" "~" (at 190.5 71.12 0)
+    (property "Reference" "#PWR0202" (at 190.5 74.93 0)
       (effects (font (size 1.27 1.27)) hide)
     )
-    (property "Datasheet" "~" (at 190.5 71.12 0)
+    (property "Value" "VCC" (at 190.5 67.31 0)
+      (effects (font (size 1.016 1.016)))
+    )
+    (property "Footprint" "" (at 190.5 71.12 0)
+      (effects (font (size 1.27 1.27)) hide)
+    )
+    (property "Datasheet" "" (at 190.5 71.12 0)
       (effects (font (size 1.27 1.27)) hide)
     )
@@
     (instances
       (project "Arduino_Uno_R3_From_Scratch"
+        (path "/e37abd6a-5ce5-42fd-a932-3d77ac2d4dc6/00000000-0000-0000-0000-000055ccfea2"
+          (reference "#PWR0202") (unit 1)
+        )
         (path "/e37abd6a-5ce5-42fd-a932-3d77ac2d4dc6/00000000-0000-0000-0000-000055d9f413"
-          (reference "#PWR025") (unit 1)
+          (reference "#PWR0301") (unit 1)
         )
       )
