File: Voltage_Regulator.kicad_sch (KiCad schematic)
At the start: 8 parts, among them CON1 BARREL_JACK, U1 LD1117S50TR

Commit message: add packages
Parts:
- C1, C2: footprint ~ -> Capacitor_SMD:C_Elec_3x5.4
- C3: footprint ~ -> Capacitor_SMD:C_0603_1608Metric
- CON1: footprint ~ -> Connector_BarrelJack:BarrelJack_Wuerth_6941xx301002
- D1: footprint ~ -> Diode_SMD:D_SMA
- D2: footprint ~ -> LED_SMD:LED_0603_1608Metric
- R1: footprint ~ -> Resistor_SMD:R_0603_1608Metric
- U1: footprint (none) -> Package_TO_SOT_SMD:TO-252-2
Changed lines of the file:
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@@
       (effects (font (size 1.016 1.016)))
     )
-    (property "Footprint" "~" (at 119.38 110.49 0)
-      (effects (font (size 1.524 1.524)))
+    (property "Footprint" "Diode_SMD:D_SMA" (at 119.38 110.49 0)
+      (effects (font (size 1.524 1.524)) hide)
     )
     (property "Datasheet" "http://www.onsemi.com/pub_link/Collateral/MRA4003T3-D.PDF" (at 119.38 110.49 0)
@@
       (effects (font (size 1.016 1.016)) (justify left))
     )
-    (property "Footprint" "~" (at 137.16 124.46 0)
-      (effects (font (size 0.762 0.762)))
+    (property "Footprint" "Capacitor_SMD:C_Elec_3x5.4" (at 137.16 124.46 0)
+      (effects (font (size 0.762 0.762)) hide)
     )
     (property "Datasheet" "http://images.ihscontent.net/vipimages/VipMasterIC/IC/BEYS/BEYSS04513/BEYSS04513-1.pdf" (at 134.62 120.65 0)
@@
       (effects (font (size 1.016 1.016)) (justify left))
     )
-    (property "Footprint" "~" (at 180.0352 124.46 0)
-      (effects (font (size 0.762 0.762)))
+    (property "Footprint" "Capacitor_SMD:C_0603_1608Metric" (at 180.0352 124.46 0)
+      (effects (font (size 0.762 0.762)) hide)
     )
     (property "Datasheet" "http://images.ihscontent.net/vipimages/VipMasterIC/IC/KEME/KEMES10043/KEMES10043-1.pdf" (at 179.07 120.65 0)
@@
       (effects (font (size 1.524 1.524)))
     )
-    (property "Footprint" "~" (at 95.25 113.03 0)
-      (effects (font (size 1.524 1.524)))
+    (property "Footprint" "Connector_BarrelJack:BarrelJack_Wuerth_6941xx301002" (at 95.25 113.03 0)
+      (effects (font (size 1.524 1.524)) hide)
     )
     (property "Datasheet" "http://katalog.we-online.de/em/datasheet/6941xx106102.pdf" (at 95.25 113.03 0)
@@
       (effects (font (size 1.524 1.524)))
     )
-    (property "Footprint" "" (at 151.13 110.49 0)
-      (effects (font (size 1.524 1.524)))
+    (property "Footprint" "Package_TO_SOT_SMD:TO-252-2" (at 151.13 110.49 0)
+      (effects (font (size 1.524 1.524)) hide)
     )
     (property "Datasheet" "http://www.st.com/st-web-ui/static/active/en/resource/technical/document/datasheet/CD00000544.pdf" (at 151.13 110.49 0)
@@
       (effects (font (size 1.016 1.016)) (justify left))
     )
-    (property "Footprint" "~" (at 171.45 124.46 0)
-      (effects (font (size 0.762 0.762)))
+    (property "Footprint" "Capacitor_SMD:C_Elec_3x5.4" (at 171.45 124.46 0)
+      (effects (font (size 0.762 0.762)) hide)
     )
     (property "Datasheet" "http://images.ihscontent.net/vipimages/VipMasterIC/IC/BEYS/BEYSS04513/BEYSS04513-1.pdf" (at 168.91 120.65 0)
@@
       (effects (font (size 1.016 1.016)))
     )
-    (property "Footprint" "~" (at 199.898 106.68 90)
-      (effects (font (size 0.762 0.762)))
+    (property "Footprint" "Resistor_SMD:R_0603_1608Metric" (at 199.898 106.68 90)
+      (effects (font (size 0.762 0.762)) hide)
     )
     (property "Datasheet" "http://www.yageo.com/pdf/Pu-RC0805_51_PbFree_L_2.pdf" (at 198.12 106.68 0)
@@
       (effects (font (size 1.27 1.27)))
     )
-    (property "Footprint" "~" (at 198.12 119.38 0)
-      (effects (font (size 1.524 1.524)))
+    (property "Footprint" "LED_SMD:LED_0603_1608Metric" (at 198.12 119.38 0)
+      (effects (font (size 1.524 1.524)) hide)
     )
     (property "Datasheet" "http://www.osram-os.com/Graphics/XPic9/00078860_0.pdf" (at 198.12 119.38 0)

Commit message: change power symbols and Arduino header
Parts:
- removed CON1: BARREL_JACK, Connector_BarrelJack:BarrelJack_Wuerth_6941xx301002, symbol Arduino_Uno_R3_From_Scratch:BARREL_JACK
- added J2: Barrel_Jack_Switch, Connector_BarrelJack:BarrelJack_Wuerth_6941xx301002, symbol Connector:Barrel_Jack_Switch
Connections:
- net GND: now also J2.2, J2.3
- net at D1.2 (A): now also J2.1
- net 5V_LDO renamed +5V
- net Vin renamed VBUS

Commit message: update power symbols
Parts:
- D1: symbol Device:D_Filled -> Device:D_Schottky_Small
- U1: footprint Package_TO_SOT_SMD:TO-252-2 -> Package_TO_SOT_SMD:SOT-223
Connections:
- net VBUS renamed VDD
