File: voltage_management.kicad_sch (KiCad schematic)
At the start: 8 parts, among them Q1 FDN340P, U2 LMV358IDGKR, U3 LP2985-33DBVR

Commit message: add packages
Parts:
- C4, C5, C6: footprint ~ -> Capacitor_SMD:C_0603_1608Metric
- Q1: footprint ~ -> Package_TO_SOT_SMD:SOT-23
- R2, R3: footprint ~ -> Resistor_SMD:R_0603_1608Metric
- U2: footprint ~ -> Package_SO:HVSSOP-8-1EP_3x3mm_P0.65mm_EP1.57x1.89mm
- U3: footprint ~ -> Package_TO_SOT_SMD:SOT-23-5
Changed lines of the file:
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@@
       (effects (font (size 1.016 1.016)))
     )
-    (property "Footprint" "~" (at 123.698 73.66 90)
-      (effects (font (size 0.762 0.762)))
+    (property "Footprint" "Resistor_SMD:R_0603_1608Metric" (at 123.698 73.66 90)
+      (effects (font (size 0.762 0.762)) hide)
     )
     (property "Datasheet" "http://images.ihscontent.net/vipimages/VipMasterIC/IC/VISH/VISHS75859/VISHS75859-1.pdf" (at 121.92 73.66 0)
@@
       (effects (font (size 1.524 1.524)) (justify right))
     )
-    (property "Footprint" "~" (at 175.26 105.41 0)
-      (effects (font (size 1.524 1.524)))
+    (property "Footprint" "Package_TO_SOT_SMD:SOT-23" (at 175.26 105.41 0)
+      (effects (font (size 1.524 1.524)) hide)
     )
     (property "Datasheet" "https://www.fairchildsemi.com/datasheets/FD/FDN340P.pdf" (at 175.26 105.41 0)
@@
       (effects (font (size 1.524 1.524)) (justify left))
     )
-    (property "Footprint" "~" (at 149.86 86.36 0)
-      (effects (font (size 1.524 1.524)))
+    (property "Footprint" "Package_SO:HVSSOP-8-1EP_3x3mm_P0.65mm_EP1.57x1.89mm" (at 149.86 86.36 0)
+      (effects (font (size 1.524 1.524)) hide)
     )
     (property "Datasheet" "http://www.ti.com/lit/ds/symlink/lmv358.pdf" (at 149.86 86.36 0)
@@
       (effects (font (size 1.524 1.524)))
     )
-    (property "Footprint" "~" (at 214.63 110.49 0)
-      (effects (font (size 1.524 1.524)))
+    (property "Footprint" "Package_TO_SOT_SMD:SOT-23-5" (at 214.63 110.49 0)
+      (effects (font (size 1.524 1.524)) hide)
     )
     (property "Datasheet" "http://www.ti.com/lit/ds/symlink/lp2985-33.pdf" (at 214.63 110.49 0)
@@
       (effects (font (size 1.016 1.016)) (justify left))
     )
-    (property "Footprint" "~" (at 230.8352 121.92 0)
-      (effects (font (size 0.762 0.762)))
+    (property "Footprint" "Capacitor_SMD:C_0603_1608Metric" (at 230.8352 121.92 0)
+      (effects (font (size 0.762 0.762)) hide)
     )
     (property "Datasheet" "http://product.tdk.com/en/catalog/datasheets/mlcc_commercial_general_en.pdf" (at 229.87 118.11 0)
@@
       (effects (font (size 1.016 1.016)) (justify left))
     )
-    (property "Footprint" "~" (at 191.4652 121.92 0)
-      (effects (font (size 0.762 0.762)))
+    (property "Footprint" "Capacitor_SMD:C_0603_1608Metric" (at 191.4652 121.92 0)
+      (effects (font (size 0.762 0.762)) hide)
     )
     (property "Datasheet" "http://www.kemet.com/docfinder?Partnumber=C0805C105K8RACAUTO" (at 190.5 118.11 0)
@@
       (effects (font (size 1.016 1.016)))
     )
-    (property "Footprint" "~" (at 123.698 93.98 90)
-      (effects (font (size 0.762 0.762)))
+    (property "Footprint" "Resistor_SMD:R_0603_1608Metric" (at 123.698 93.98 90)
+      (effects (font (size 0.762 0.762)) hide)
     )
     (property "Datasheet" "http://images.ihscontent.net/vipimages/VipMasterIC/IC/VISH/VISHS75859/VISHS75859-1.pdf" (at 121.92 93.98 0)
@@
       (effects (font (size 1.016 1.016)) (justify left))
     )
-    (property "Footprint" "~" (at 88.9 72.0852 0)
-      (effects (font (size 0.762 0.762)))
+    (property "Footprint" "Capacitor_SMD:C_0603_1608Metric" (at 88.9 72.0852 0)
+      (effects (font (size 0.762 0.762)) hide)
     )
     (property "Datasheet" "http://images.ihscontent.net/vipimages/VipMasterIC/IC/KEME/KEMES10043/KEMES10043-1.pdf" (at 92.71 71.12 0)
@@
       (effects (font (size 1.524 1.524)) (justify left))
     )
-    (property "Footprint" "~" (at 85.09 87.63 0)
-      (effects (font (size 1.524 1.524)))
+    (property "Footprint" "Package_SO:HVSSOP-8-1EP_3x3mm_P0.65mm_EP1.57x1.89mm" (at 85.09 87.63 0)
+      (effects (font (size 1.524 1.524)) hide)
     )
     (property "Datasheet" "http://www.ti.com/lit/ds/symlink/lmv358.pdf" (at 85.09 87.63 0)

Commit message: change power symbols and Arduino header
Connections:
- net 5V_LDO renamed +5V
- net USBVCC renamed VCC
- net Vin renamed VBUS
Changed lines of the file:
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@@
     )
   )
-  (symbol (lib_id "Arduino_Uno_R3_From_Scratch:USBVCC") (at 165.1 104.14 0) (unit 1)
+  (symbol (lib_id "power:VCC") (at 165.1 104.14 0) (unit 1)
     (in_bom yes) (on_board yes) (dnp no)
     (property "Reference" "#PWR012" (at 165.1 101.854 0)
@@
     )
     (property "Footprint" "~" (at 165.1 104.14 0)
-      (effects (font (size 1.524 1.524)))
+      (effects (font (size 1.27 1.27)) hide)
     )
     (property "Datasheet" "~" (at 165.1 104.14 0)
-      (effects (font (size 1.524 1.524)))
+      (effects (font (size 1.27 1.27)) hide)
     )
     (pin "1")
@@
     )
   )
-  (symbol (lib_id "Arduino_Uno_R3_From_Scratch:5V_LDO") (at 184.15 95.25 0) (unit 1)
+  (symbol (lib_id "power:+5V") (at 184.15 95.25 0) (unit 1)
     (in_bom yes) (on_board yes) (dnp no)
     (property "Reference" "#PWR014" (at 184.15 92.964 0)
@@
     )
     (property "Footprint" "~" (at 184.15 95.25 0)
-      (effects (font (size 1.524 1.524)))
+      (effects (font (size 1.27 1.27)) hide)
     )
     (property "Datasheet" "~" (at 184.15 95.25 0)
-      (effects (font (size 1.524 1.524)))
+      (effects (font (size 1.27 1.27)) hide)
     )
     (pin "1")
@@
     )
   )
-  (symbol (lib_id "Arduino_Uno_R3_From_Scratch:5V_LDO") (at 82.55 64.77 0) (unit 1)
+  (symbol (lib_id "power:+5V") (at 82.55 64.77 0) (unit 1)
     (in_bom yes) (on_board yes) (dnp no)
     (property "Reference" "#PWR015" (at 82.55 62.484 0)
@@
     )
     (property "Footprint" "~" (at 82.55 64.77 0)
-      (effects (font (size 1.524 1.524)))
+      (effects (font (size 1.27 1.27)) hide)
     )
     (property "Datasheet" "~" (at 82.55 64.77 0)
-      (effects (font (size 1.524 1.524)))
+      (effects (font (size 1.27 1.27)) hide)
     )
     (pin "1")
@@
     )
   )
-  (symbol (lib_id "Arduino_Uno_R3_From_Scratch:Vin") (at 121.92 64.77 0) (unit 1)
+  (symbol (lib_id "power:VBUS") (at 121.92 64.77 0) (unit 1)
     (in_bom yes) (on_board yes) (dnp no)
     (property "Reference" "#PWR016" (at 121.92 62.484 0)
@@
     )
     (property "Footprint" "~" (at 121.92 64.77 0)
-      (effects (font (size 1.524 1.524)))
+      (effects (font (size 1.27 1.27)) hide)
     )
     (property "Datasheet" "~" (at 121.92 64.77 0)
-      (effects (font (size 1.524 1.524)))
-    )
-    (pin "1")
+      (effects (font (size 1.27 1.27)) hide)
+    )
+    (pin "1")

Commit message: update power symbols
Connections:
- net 3V3_LDO renamed +3V3
- net VBUS renamed VDD
