File: Arduino_Uno_R3_From_Scratch.kicad_pcb (KiCad board)
At the start: 2 copper layers, 59 parts, among them CON1 BARREL_JACK, J1 USB_TYPE_B, P1 Power Header, P2 Analog Header, P3 Digital Header 02, P4 Digital Header 01, Q1 FDN340P, SW1 RESET_SWITCH, U1 LD1117S50TR, U2 LMV358IDGKR, U3 LP2985-33DBVR, U4 ATMEGA16U2-MU, U5 ATMEGA328P, X1 FOXSLF/160-20, X2 CSTCE16MOV53-R0

Commit message: initial PCB layout
Parts:
- removed CON1: BARREL_JACK, Connector_BarrelJack:BarrelJack_Wuerth_6941xx301002
- removed ICSP2: M20-9980346, Connector_PinHeader_2.54mm:PinHeader_2x03_P2.54mm_Vertical
- removed P1: Power Header, Connector_PinSocket_2.54mm:PinSocket_1x08_P2.54mm_Vertical
- removed P2: Analog Header, Connector_PinSocket_2.54mm:PinSocket_1x06_P2.54mm_Vertical
- removed P3: Digital Header 02, Connector_PinSocket_2.54mm:PinSocket_1x10_P2.54mm_Vertical
- removed P4: Digital Header 01, Connector_PinSocket_2.54mm:PinSocket_1x08_P2.54mm_Vertical
- added J2: Barrel_Jack_Switch, Connector_BarrelJack:BarrelJack_Wuerth_6941xx301002, F.Cu at (121.1, 116.1)
- added XA1: Arduino_Uno_R3_SMD_Shield, User Custom Footprint:Arduino_Uno_R3_MountingHole, F.Cu at (110.4, 123.8)
- J1: footprint Connector_USB:USB_B_Lumberg_2411_02_Horizontal -> Connector_USB:USB_Micro-B_Molex-105017-0001
- moved R14 145.6 mm to (165.1, 107.0)
- moved R15 145.6 mm to (165.1, 109.5)
- moved R16 142.0 mm to (165.0, 103.6)
- moved R17 140.1 mm to (165.4, 100.3)
- moved C14 136.3 mm to (148.1, 108.0)
- moved R12 135.7 mm to (148.3, 111.5)
- moved C11 135.6 mm to (148.3, 103.9)
- moved U5 135.4 mm to (156.7, 107.2), turned to 180 degrees
- moved X2 134.9 mm to (161.7, 95.7), turned to -90 degrees
- moved D7 132.0 mm to (170.2, 96.0), turned to 90 degrees
- moved C15 131.4 mm to (148.3, 100.8)
- moved R13 123.0 mm to (142.2, 99.6)
- moved R1 104.2 mm to (173.2, 83.3)
- moved D2 102.2 mm to (173.2, 80.8)
- moved C2 98.3 mm to (140.0, 116.1)
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- renumbered MF-MSMF050-2 to F1
Connections:
- net 328P_ICSP_SCK renamed /ATMEGA328P/ARD_DIG13/SPI_SCK
- net USBVCC renamed VCC
- net Vin renamed VBUS
- C15 pad 1: 5V_LDO -> +5V
- C2 pad 1: 5V_LDO -> +5V
- C3 pad 1: 5V_LDO -> +5V
- C4 pad 2: 5V_LDO -> +5V
- C5 pad 1: 5V_LDO -> +5V
- C9 pad 1: 5V_LDO -> +5V
- D4 pad 2: 5V_LDO -> +5V
- D7 pad 1: /ATMEGA328P/328P_RESET -> +5V
- D7 pad 2: 5V_LDO -> +5V
- FB1 pad 1: Net-(J1-Shield_1) -> Net-(J1-Shield)
- ICSP1 pad 2: 5V_LDO -> +5V
- J1 pad 4: /ATMEGA16U2/USB_GND -> unconnected-(J1-ID-Pad4)
- J1 pad 5: Net-(J1-Shield_1) -> /ATMEGA16U2/USB_GND
- Q1 pad 2: 5V_LDO -> +5V
- R1 pad 2: 5V_LDO -> +5V
- R10 pad 2: 5V_LDO -> +5V
- R11 pad 2: 5V_LDO -> +5V
- R13 pad 2: /ATMEGA328P/328P_RESET -> +5V
- R16 pad 1: /ATMEGA328P/328P_RESET -> +5V
- R16 pad 2: 5V_LDO -> +5V
- R5 pad 1: Net-(J1-D-) -> Net-(J1-D+)
- R6 pad 1: Net-(J1-D+) -> Net-(J1-D-)
- R7 pad 2: 5V_LDO -> +5V
- U1 pad 2: 5V_LDO -> +5V
- U2 pad 8: 5V_LDO -> +5V
- U3 pad 1: 5V_LDO -> +5V
- U3 pad 3: 5V_LDO -> +5V
- U4 pad 32: 5V_LDO -> +5V
- U4 pad 4: 5V_LDO -> +5V
- U5 pad 1: /ATMEGA328P/328P_RESET -> +5V
- U5 pad 17: 328P_ICSP_MOSI -> /ATMEGA328P/ARD_DIG11/SPI_MOSI
- U5 pad 18: 328P_ICSP_MISO -> /ATMEGA328P/ARD_DIG12/SPI_MISO
- U5 pad 20: 5V_LDO -> +5V
- U5 pad 7: 5V_LDO -> +5V
- VR1 pad 1: Net-(J1-D+) -> Net-(J1-D-)
- VR1 pad 2: Net-(J1-Shield_1) -> Net-(J1-Shield)
- VR2 pad 1: Net-(J1-D-) -> Net-(J1-D+)
- VR2 pad 2: Net-(J1-Shield_1) -> Net-(J1-Shield)
Other:
- board outline added: 68.6 x 53.3 mm

Commit message: update pcb to 4 layers
- update PCB to 4 layers
- add 3d models of pin sockets to Arduino board
- update net color
- add ground/power planes (inner layers)
Parts:
- removed R7: 10K, Resistor_SMD:R_0603_1608Metric
- U1: footprint Package_TO_SOT_SMD:TO-252-2 -> Package_TO_SOT_SMD:SOT-223
- moved F1 18.5 mm to (113.0, 80.3)
- moved C15 15.0 mm to (162.9, 104.0), turned to 90 degrees
- moved R16 7.75 mm to (165.4, 111.4)
- moved R4 2.99 mm to (135.5, 103.8)
- moved R14 2.90 mm to (165.4, 109.9), turned to 180 degrees
- moved D4 2.53 mm to (116.0, 97.5)
- moved U1 1.81 mm to (116.3, 104.9)
- moved D3 1.70 mm to (135.6, 100.6)
- moved Q1 1.52 mm to (130.4, 109.3)
- moved R15 1.17 mm to (165.4, 108.3), turned to 180 degrees
- moved U2 1.00 mm to (130.8, 103.8)
- moved D7 0.52 mm to (169.7, 95.9)
Connections:
- net VBUS renamed VDD
- C6 pad 1: 3V3_LDO -> +3V3
- D7 pad 2: +5V -> Net-(D7-A)
- R13 pad 2: +5V -> /ATMEGA328P/328P_RESET
- R16 pad 1: +5V -> /ATMEGA328P/328P_RESET
- U2 pad 2: 3V3_LDO -> +3V3
- U3 pad 5: 3V3_LDO -> +3V3
- U5 pad 1: +5V -> /ATMEGA328P/328P_RESET
- XA1 pad 3V3: +3.3V -> +3V3
- XA1 pad 5V2: +5V -> Net-(D7-A)
- XA1 pad RST1: +5V -> /ATMEGA328P/328P_RESET
- XA1 pad RST2: +5V -> /ATMEGA328P/328P_RESET
Routing:
- net Net-(U2B--): track 0.00 -> 3.03 mm
- added copper zone on In2.Cu, net +5V
- added copper zone on In1.Cu, net GND
Other:
- copper layers 2 -> 4
